File: pcb/rp2040.kicad_sch (KiCad schematic)
At the start: 26 parts, among them P1 USB_C_Plug_USB2.0, SW44 SW_Push, U1 RP2040, U2 NCP1117-3.3_SOT223, U3 W25Q128JVS, Y1 ABM8-272-T3

Commit message: add pcb stuff
Parts:
- removed P1: USB_C_Plug_USB2.0, Connector_USB:USB_C_Receptacle_GCT_USB4125-xx-x-0190_6P_TopMnt_Horizontal, symbol Connector:USB_C_Plug_USB2.0
- added J1: USB_C_Receptacle_USB2.0_16P, Connector_USB:USB_C_Receptacle_HCTL_HC-TYPE-C-16P-01A, symbol Connector:USB_C_Receptacle_USB2.0_16P
- added R5, R6: 5.1k, Resistor_SMD:R_0402_1005Metric, symbol Device:R_Small
- C14: value C_Small -> 100n
Connections:
- net GND: now also J1.A1 (GND), J1.A12 (GND), J1.B1 (GND), J1.B12 (GND), J1.S1 (SHIELD), R5.2, R6.2
- net USB_D+: now also J1.A6 (D+), J1.B6 (D+)
- net USB_D-: now also J1.A7 (D-), J1.B7 (D-)
- net VBUS: now also J1.A4 (VBUS), J1.A9 (VBUS), J1.B4 (VBUS), J1.B9 (VBUS)
- new net: J1.B5 (CC2), R6.1
- new net: J1.A5 (CC1), R5.1
Other:
- moved on the sheet: C1, C2, U2

Commit message: add firmware
Parts:
- added J2: Conn_01x04, Connector_PinHeader_2.54mm:PinHeader_1x04_P2.54mm_Vertical, symbol Connector_Generic:Conn_01x04
Connections:
- net GND: now also J2.3 (Pin_3)
- net SWCLK: now reaches U1.24 (SWCLK)
- net SWCLK: now also J2.2 (Pin_2)
- net SWD: now reaches U1.25 (SWD)
- net SWD: now also J2.1 (Pin_1)
- net RUN: now reaches U1.26 (RUN)
- net RUN: now also J2.4 (Pin_4)
- no-connect marks 18 -> 16
