File: pcb/steno.kicad_pcb (KiCad board)
At the start: 2 copper layers, 268.7 x 76.2 mm, 119 parts, among them P1 USB_C_Plug_USB2.0, SW1 SW_Push_45deg, SW10 SW_Push_45deg, SW11 SW_Push_45deg, SW12 SW_Push_45deg, SW13 SW_Push_45deg, SW14 SW_Push_45deg, SW15 SW_Push_45deg, SW16 SW_Push_45deg, SW17 SW_Push_45deg, SW18 SW_Push_45deg, SW19 SW_Push_45deg, SW2 SW_Push_45deg, SW20 SW_Push_45deg, SW21 SW_Push_45deg, SW22 SW_Push_45deg, SW23 SW_Push_45deg, SW24 SW_Push_45deg, SW25 SW_Push_45deg, SW26 SW_Push_45deg, SW27 SW_Push_45deg, SW28 SW_Push_45deg, SW29 SW_Push_45deg, SW3 SW_Push_45deg, SW31 SW_Push_45deg, SW32 SW_Push_45deg, SW33 SW_Push_45deg, SW34 SW_Push_45deg, SW35 SW_Push_45deg, SW36 SW_Push_45deg, SW37 SW_Push_45deg, SW38 SW_Push_45deg, SW39 SW_Push_45deg, SW4 SW_Push_45deg, SW40 SW_Push_45deg, SW41 SW_Push_45deg, SW42 SW_Push_45deg, SW43 SW_Push_45deg, SW44 SW_Push, SW5 SW_Push_45deg, SW6 SW_Push_45deg, SW7 SW_Push_45deg, SW8 SW_Push_45deg, SW9 SW_Push_45deg, U1 RP2040, U2 NCP1117-3.3_SOT223, U3 W25Q128JVS, Y1 ABM8-272-T3

Commit message: add pcb stuff
Parts:
- removed P1: USB_C_Plug_USB2.0, Connector_USB:USB_C_Receptacle_GCT_USB4125-xx-x-0190_6P_TopMnt_Horizontal
- added J1: USB_C_Receptacle_USB2.0_16P, Connector_USB:USB_C_Receptacle_HCTL_HC-TYPE-C-16P-01A, F.Cu at (158.1, 34.5)
- added R5: 5.1k, Resistor_SMD:R_0402_1005Metric, F.Cu at (160.0, 42.6)
- added R6: 5.1k, Resistor_SMD:R_0402_1005Metric, F.Cu at (157.9, 42.6)
- moved U2 4.37 mm to (158.1, 49.4)
- moved C1 2.95 mm to (155.8, 42.6)
Routing:
- net /rp2040/USB_D-: track 0.00 -> 28.5 mm, vias 0 -> 2
- net /rp2040/USB_D+: track 0.00 -> 24.8 mm, vias 0 -> 2
- net VBUS: track 10.0 -> 16.4 mm
- net R0: track 300.3 -> 306.7 mm
- net Net-(J1-CC2): track 0.00 -> 4.78 mm
- net Net-(J1-CC1): track 0.00 -> 4.43 mm
- net +3V3: track 63.1 -> 58.7 mm

Commit message: add firmware
Parts:
- added J2: Conn_01x04, Connector_PinHeader_2.54mm:PinHeader_1x04_P2.54mm_Vertical, F.Cu at (143.7, 70.0)
- C14: value C_Small -> 100n
- moved C5 1.13 mm to (161.5, 73.6)
- moved C4 0.48 mm to (160.4, 73.0)
Connections:
- U1 pad 24: unconnected-(U1-SWCLK-Pad24) -> /rp2040/SWCLK
- U1 pad 25: unconnected-(U1-SWD-Pad25) -> /rp2040/SWD
- U1 pad 26: unconnected-(U1-RUN-Pad26) -> /rp2040/RUN
Routing:
- net /rp2040/SWCLK: track 0.00 -> 49.1 mm, vias 0 -> 8
- net /rp2040/SWD: track 0.00 -> 47.5 mm, vias 0 -> 3
- net /rp2040/RUN: track 0.00 -> 39.6 mm, vias 0 -> 3
- net +1V1: track 18.9 -> 39.6 mm, vias 3 -> 5
- net C10: track 160.4 -> 168.8 mm
- net C11: track 173.2 -> 177.2 mm
- net R1: track 289.1 -> 291.7 mm
- net GND: track 38.4 -> 39.8 mm, vias 20 -> 10
- net R2: track 260.8 -> 261.8 mm
